Commit message: _

File: src/unitree_robot_description/urdf/hardware_driver/unitree_arm_ros2_control.xacro (robot description, xacro)
@@ -25,4 +25,13 @@
                 <state_interface name="effort"/>
             </joint>
+            <joint name="joint3">
+                <param name="motor_id">2</param>
+                <command_interface name="position"/>
+                <command_interface name="velocity"/>
+                <command_interface name="effort"/>
+                <state_interface name="position"/>
+                <state_interface name="velocity"/>
+                <state_interface name="effort"/>
+            </joint>
         </ros2_control>
     </xacro:macro>

File: src/unitree_robot_description/urdf/mock_components/mock_arm_ros2_control.xacro (robot description, xacro)
@@ -23,4 +23,12 @@
                 <state_interface name="effort"/>
             </joint>
+            <joint name="joint3">
+                <command_interface name="position"/>
+                <command_interface name="velocity"/>
+                <command_interface name="effort"/>
+                <state_interface name="position"/>
+                <state_interface name="velocity"/>
+                <state_interface name="effort"/>
+            </joint>
         </ros2_control>
     </xacro:macro>

File: src/unitree_robot_description/urdf/unitree_arm_description.xacro (robot description, xacro)
@@ -9,4 +9,6 @@
     <xacro:property name="link2_length" value="0.2"/>
     <xacro:property name="link2_radius" value="0.025"/>
+    <xacro:property name="link3_length" value="0.15"/>
+    <xacro:property name="link3_radius" value="0.02"/>
     <material name="grey">
         <color rgba="0.7 0.7 0.7 1.0"/>
@@ -17,4 +19,7 @@
     <material name="yellow">
         <color rgba="1.0 1.0 0.0 1.0"/>
+    </material>
+    <material name="blue">
+        <color rgba="0.0 0.3 1.0 1.0"/>
     </material>
     <xacro:macro name="unitree_arm_description">
@@ -87,4 +92,29 @@
             </xacro:inertial_cylinder>
         </link>
+        <joint name="joint3" type="revolute">
+            <parent link="link2"/>
+            <child link="link3"/>
+            <origin xyz="0 0 ${link2_length}" rpy="0 0 0"/>
+            <axis xyz="0 1 0"/>
+            <limit lower="-2.0" upper="2.0" effort="30.0" velocity="10.0"/>
+        </joint>
+        <link name="link3">
+            <visual>
+                <origin xyz="0 0 ${link3_length/2}" rpy="0 0 0"/>
+                <geometry>
+                    <cylinder radius="${link3_radius}" length="${link3_length}"/>
+                </geometry>
+                <material name="blue"/>
+            </visual>
+            <collision>
+                <origin xyz="0 0 ${link3_length/2}" rpy="0 0 0"/>
+                <geometry>
+                    <cylinder radius="${link3_radius}" length="${link3_length}"/>
+                </geometry>
+            </collision>
+            <xacro:inertial_cylinder mass="0.3" length="${link3_length}" radius="${link3_radius}">
+                <origin xyz="0 0 ${link3_length/2}" rpy="0 0 0"/>
+            </xacro:inertial_cylinder>
+        </link>
     </xacro:macro>
 </robot>
